Commit message: Spencer (modified) working in simulation

File: base_simulation/urdf/iliad_uol_cititruck.xacro (robot description, xacro)
@@ -5,4 +5,10 @@
     <xacro:arg name="kinect2" default="false"/>
     <xacro:arg name="kinect1" default="false"/> <!-- deprecated -->
+    <!-- Arguments used in cititruck.gazebo -->
+    <xacro:arg name="controller_prefix" default=""/>
+    <xacro:arg name="sensor_prefix" default=""/>
+    <xacro:arg name="sick_name" default="safety"/>
+    <xacro:arg name="ls2000_name" default="nav"/>
+    <xacro:arg name="kinect2_name" default=""/>
     <!-- Import all Gazebo-customization elements, including Gazebo colors -->
     <xacro:include filename="$(find cititruck_description)/urdf/cititruck.gazebo"/>
@@ -42,25 +48,26 @@
             <material name="red"/>
         </visual>
-        <!-- Top shelf -->
-        <visual>
-            <origin xyz="0.8 0 1.1" rpy="0 0 0" />
-            <geometry>
-                <box size="0.4 0.55 0.03" />
-            </geometry>
-            <material name="red"/>
-        </visual>
-        <visual>
-            <origin xyz="0.985 0.26 0.9" rpy="0 0 0" />
-            <geometry>
-                <box size="0.03 0.03 0.4" />
-            </geometry>
-            <material name="red"/>
-        </visual>
-        <visual>
-            <origin xyz="0.985 -0.26 0.9" rpy="0 0 0" />
-            <geometry>
-                <box size="0.03 0.03 0.4" />
-            </geometry>
-            <material name="red"/>
+        <!-- Top Bar -->
+        <visual>
+            <origin xyz="0.8 0 0.935" rpy="0 0 0" />
+            <geometry>
+                <!-- box size="0.4 0.55 0.03" / -->
+                <box size="0.05 0.54 0.025" />
+            </geometry>
+            <material name="gray"/>
+        </visual>
+        <visual>
+            <origin xyz="0.8 0.26 0.85" rpy="0 0 0" />
+            <geometry>
+                <box size="0.05 0.025 0.18" />
+            </geometry>
+            <material name="gray"/>
+        </visual>
+        <visual>
+            <origin xyz="0.8 -0.26 0.85" rpy="0 0 0" />
+            <geometry>
+                <box size="0.05 0.025 0.18" />
+            </geometry>
+            <material name="gray"/>
         </visual>
     </link>
@@ -281,5 +288,5 @@
     <!-- SENSORS START HERE -->
     <!-- SICK laser -->
-    <link name="safety_laser_link">
+    <link name="$(arg sick_name)_link">
         <collision>
             <origin xyz="0 0 0" rpy="0 0 0"/>
@@ -300,12 +307,12 @@
         </inertial>
     </link>
-    <joint name="safety_laser_joint" type="fixed">
+    <joint name="$(arg sick_name)_joint" type="fixed">
         <axis xyz="0 1 0"/>
         <origin xyz="1.4 0 0.02" rpy="3.14159 0 0"/>
         <parent link="base_link"/>
-        <child link="safety_laser_link"/>
+        <child link="$(arg sick_name)_link"/>
     </joint>
     <!-- LS2000 navigation/localization laser -->
-    <link name="nav_laser_link">
+    <link name="$(arg ls2000_name)_link">
         <collision>
             <origin xyz="0 0 0" rpy="0 0 0"/>
@@ -326,13 +333,13 @@
         </inertial>
     </link>
-    <joint name="nav_laser_joint" type="fixed">
+    <joint name="$(arg ls2000_name)_joint" type="fixed">
         <origin xyz="0.8 0 0.85" rpy="0 0 0"/>
         <parent link="base_link"/>
-        <child link="nav_laser_link"/>
+        <child link="$(arg ls2000_name)_link"/>
     </joint>
     <!-- Velodyne VLP16 -->
     <xacro:if value="$(arg velodyne)">
-      <xacro:include filename="$(find velodyne_description)/urdf/VLP-16.urdf.xacro"/>
-      <VLP-16 parent="base_link" prefix="$(arg tf_prefix)" name="velodyne" topic="/velodyne_points" hz="10" samples="440">
+      <xacro:include filename="$(find velodyne_description8)/urdf/VLP-16.urdf.xacro"/>
+      <VLP-16 parent="base_link" gpu="true" name="$(arg tf_prefix)/velodyne" topic="/$(arg tf_prefix)/$(arg sensor_prefix)/velodyne/velodyne_points" hz="10" samples="440">
           <origin xyz="0.8 0 0.95" rpy="0 0 0" />
       </VLP-16>
@@ -340,6 +347,6 @@
     <!-- Kinect v2 -->
     <xacro:if value="$(arg kinect2)">
-      <xacro:include filename="$(find kinect2_description)/urdf/kinect2/kinect2.xacro"/>
-      <kinect2_sensor parent="base_link" prefix="$(arg tf_prefix)" name="kinect2" cam_px="0.98" cam_py="0" cam_pz="1.15" cam_or="0" cam_op="0" cam_oy="0"/>
+      <xacro:include filename="$(find base_simulation)/urdf/kinect2b.xacro"/>
+      <kinect2_sensor parent="base_link" prefix="/$(arg tf_prefix)/$(arg sensor_prefix)/kinect2" name="kinect2" cam_px="0.8" cam_py="0" cam_pz="1.05" cam_or="0" cam_op="0" cam_oy="0.0"/>
     </xacro:if>
     <!-- Old Kinect (deprecated, only used for pallet detection?) -->

Commit message: calibrated xacro

File: base_simulation/urdf/iliad_uol_cititruck.xacro (robot description, xacro)
@@ -4,5 +4,5 @@
     <xacro:arg name="velodyne" default="false"/>
     <xacro:arg name="kinect2" default="false"/>
-    <xacro:arg name="kinect1" default="false"/> <!-- deprecated -->
+    <xacro:arg name="asus" default="false"/> <!-- not used by Cititruck? -->
     <!-- Arguments used in cititruck.gazebo -->
     <xacro:arg name="controller_prefix" default=""/>
@@ -10,9 +10,13 @@
     <xacro:arg name="sick_name" default="safety"/>
     <xacro:arg name="ls2000_name" default="nav"/>
-    <xacro:arg name="kinect2_name" default=""/>
+    <xacro:arg name="kinect2_name" default="kinect2"/>
+    <xacro:arg name="asus_name" default="asus"/>
+    <xacro:arg name="is_uol_variant" default="true"/>
     <!-- Import all Gazebo-customization elements, including Gazebo colors -->
     <xacro:include filename="$(find cititruck_description)/urdf/cititruck.gazebo"/>
     <!-- Import Rviz colors -->
     <xacro:include filename="$(find cititruck_description)/urdf/materials.xacro"/>
+    <!-- Adds extra joints for calibration of sensors -->
+    <xacro:include filename="$(find cititruck_description)/urdf/sensor_calibration_assembly.xacro" />
     <xacro:property name="forks_pidP" value="2000"/>
     <xacro:property name="forks_pidI" value="0"/>
@@ -48,5 +52,30 @@
             <material name="red"/>
         </visual>
-        <!-- Top Bar -->
+	<!-- Top shelf ORU version -->
+    <xacro:unless value="$(arg is_uol_variant)">
+        <visual>
+            <origin xyz="0.8 0 1.1" rpy="0 0 0" />
+            <geometry>
+                <box size="0.4 0.55 0.03" />
+            </geometry>
+            <material name="red"/>
+        </visual>
+        <visual>
+            <origin xyz="0.985 0.26 0.9" rpy="0 0 0" />
+            <geometry>
+                <box size="0.03 0.03 0.4" />
+            </geometry>
+            <material name="red"/>
+        </visual>
+        <visual>
+            <origin xyz="0.985 -0.26 0.9" rpy="0 0 0" />
+            <geometry>
+                <box size="0.03 0.03 0.4" />
+            </geometry>
+            <material name="red"/>
+        </visual>
+    </xacro:unless>
+    <!-- Top Bar UoL version -->
+    <xacro:if value="$(arg is_uol_variant)">
         <visual>
             <origin xyz="0.8 0 0.935" rpy="0 0 0" />
@@ -71,4 +100,5 @@
             <material name="gray"/>
         </visual>
+    </xacro:if>
     </link>
     <!-- Forks -->
@@ -288,5 +318,5 @@
     <!-- SENSORS START HERE -->
     <!-- SICK laser -->
-    <link name="$(arg sick_name)_link">
+    <link name="$(arg sick_name)_base_link">
         <collision>
             <origin xyz="0 0 0" rpy="0 0 0"/>
@@ -311,8 +341,9 @@
         <origin xyz="1.4 0 0.02" rpy="3.14159 0 0"/>
         <parent link="base_link"/>
-        <child link="$(arg sick_name)_link"/>
-    </joint>
+        <child link="$(arg sick_name)_base_link"/>
+    </joint>
+    <sensor_calibration_assembly sensor_id="$(arg sick_name)" parent_link="$(arg sick_name)_base_link"/>
     <!-- LS2000 navigation/localization laser -->
-    <link name="$(arg ls2000_name)_link">
+    <link name="$(arg ls2000_name)_base_link">
         <collision>
             <origin xyz="0 0 0" rpy="0 0 0"/>
@@ -336,21 +367,26 @@
         <origin xyz="0.8 0 0.85" rpy="0 0 0"/>
         <parent link="base_link"/>
-        <child link="$(arg ls2000_name)_link"/>
-    </joint>
+        <child link="$(arg ls2000_name)_base_link"/>
+    </joint>
+    <sensor_calibration_assembly sensor_id="$(arg ls2000_name)" parent_link="$(arg ls2000_name)_base_link"/>
     <!-- Velodyne VLP16 -->
+    <!-- FIXME: We should rather attach the calibration assembly to the final link, otherwise we have a 3.7cm z offset during rotation, so need to split up the imported xacro -->
+    <!-- FIXED: The name should be velodyne_link -->
     <xacro:if value="$(arg velodyne)">
-      <xacro:include filename="$(find velodyne_description8)/urdf/VLP-16.urdf.xacro"/>
-      <VLP-16 parent="base_link" gpu="true" name="velodyne" topic="/$(arg tf_prefix)/$(arg sensor_prefix)/velodyne/velodyne_points" hz="10" samples="440">
-          <origin xyz="0.8 0 0.95" rpy="0 0 0" />
+      <xacro:include filename="$(find velodyne_description)/urdf/VLP-16.urdf.xacro"/>
+      <VLP-16 parent="velodyne_base_link" prefix="$(arg tf_prefix)" name="velodyne_link" topic="$(arg sensor_prefix)/velodyne_points" hz="10" samples="440">
+          <origin xyz="0 0 0" rpy="0 0 0" /> <!-- given by calibration -->
       </VLP-16>
+      <sensor_calibration_assembly sensor_id="velodyne" parent_link="base_link" final_link_suffix="base_link"/>
     </xacro:if>
     <!-- Kinect v2 -->
     <xacro:if value="$(arg kinect2)">
-      <xacro:include filename="$(find base_simulation)/urdf/kinect2b.xacro"/>
-      <kinect2_sensor parent="base_link" prefix="/$(arg tf_prefix)/$(arg sensor_prefix)/kinect2" name="kinect2" cam_px="0.8" cam_py="0" cam_pz="1.05" cam_or="0" cam_op="0" cam_oy="0.0"/>
+      <xacro:include filename="$(find kinect2_description)/urdf/kinect2/kinect2.xacro"/>
+      <kinect2_sensor parent="kinect2_base_link" prefix="$(arg tf_prefix)/$(arg sensor_prefix)" name="kinect2" cam_px="0" cam_py="0" cam_pz="0" cam_or="0" cam_op="0" cam_oy="3.1415926"/>
+      <sensor_calibration_assembly sensor_id="kinect2" parent_link="base_link" final_link_suffix="base_link"/>
     </xacro:if>
-    <!-- Old Kinect (deprecated, only used for pallet detection?) -->
-    <xacro:if value="$(arg kinect1)">
-      <link name="kinect_link">
+    <!-- Asus for pallet detection (deprecated?) -->
+    <xacro:if value="$(arg asus)">
+      <link name="$(arg asus_name)_base_link">
           <collision>
               <origin xyz="0 0 0" rpy="0 0 0"/>
@@ -371,11 +407,12 @@
           </inertial>
       </link>
-      <joint name="kinect_joint" type="fixed">
+      <joint name="$(arg asus_name)_joint" type="fixed">
           <axis xyz="0 1 0"/>
           <origin xyz="0.5 0 0.7" rpy="0 2.5 0"/> <!-- 0 2.5 0 -->
           <!--        <origin xyz="0.5 0 0.7" rpy="0 3.14159 0"/>-->
           <parent link="base_link"/>
-          <child link="kinect_link"/>
+          <child link="$(arg asus_name)_base_link"/>
       </joint>
+      <sensor_calibration_assembly sensor_id="$(arg asus_name)" parent_link="$(arg asus_name)_base_link"/>
     </xacro:if>
 </robot>

Commit message: WIP: correcting tf tree

File: base_simulation/urdf/iliad_uol_cititruck.xacro (robot description, xacro)
@@ -374,9 +374,9 @@
     <!-- FIXED: The name should be velodyne_link -->
     <xacro:if value="$(arg velodyne)">
-      <xacro:include filename="$(find velodyne_description)/urdf/VLP-16.urdf.xacro"/>
-      <VLP-16 parent="velodyne_base_link" prefix="$(arg tf_prefix)" name="velodyne_link" topic="$(arg sensor_prefix)/velodyne_points" hz="10" samples="440">
-          <origin xyz="0 0 0" rpy="0 0 0" /> <!-- given by calibration -->
+      <xacro:include filename="$(find velodyne_description8)/urdf/VLP-16.urdf.xacro"/>
+      <VLP-16 parent="velodyne_base_link" gpu="true" name="velodyne_link" topic="/$(arg tf_prefix)/$(arg sensor_prefix)/velodyne/velodyne_points" hz="10" samples="440">
+          <origin xyz="0.8 0 0.95" rpy="0 0 0" />
       </VLP-16>
-      <sensor_calibration_assembly sensor_id="velodyne" parent_link="base_link" final_link_suffix="base_link"/>
+     <sensor_calibration_assembly sensor_id="velodyne" parent_link="base_link" final_link_suffix="base_link"/>
     </xacro:if>
     <!-- Kinect v2 -->

Commit message: Final corrections in tfs. Asus model works now like kinect2 model. Velodyne name corrected.

File: base_simulation/urdf/iliad_uol_cititruck.xacro (robot description, xacro)
@@ -375,5 +375,5 @@
     <xacro:if value="$(arg velodyne)">
       <xacro:include filename="$(find velodyne_description8)/urdf/VLP-16.urdf.xacro"/>
-      <VLP-16 parent="velodyne_base_link" gpu="true" name="velodyne_link" topic="/$(arg tf_prefix)/$(arg sensor_prefix)/velodyne/velodyne_points" hz="10" samples="440">
+      <VLP-16 parent="velodyne_base_link" gpu="true" name="velodyne" topic="/$(arg tf_prefix)/$(arg sensor_prefix)/velodyne/velodyne_points" hz="10" samples="440">
           <origin xyz="0.8 0 0.95" rpy="0 0 0" />
       </VLP-16>
@@ -382,37 +382,13 @@
     <!-- Kinect v2 -->
     <xacro:if value="$(arg kinect2)">
-      <xacro:include filename="$(find kinect2_description)/urdf/kinect2/kinect2.xacro"/>
+    <xacro:include filename="$(find kinect2_description)/urdf/kinect2/kinect2.xacro"/>
       <kinect2_sensor parent="kinect2_base_link" prefix="$(arg tf_prefix)/$(arg sensor_prefix)" name="kinect2" cam_px="0" cam_py="0" cam_pz="0" cam_or="0" cam_op="0" cam_oy="3.1415926"/>
       <sensor_calibration_assembly sensor_id="kinect2" parent_link="base_link" final_link_suffix="base_link"/>
     </xacro:if>
-    <!-- Asus for pallet detection (deprecated?) -->
+    <!-- Asus for pallet detection -->
     <xacro:if value="$(arg asus)">
-      <link name="$(arg asus_name)_base_link">
-          <collision>
-              <origin xyz="0 0 0" rpy="0 0 0"/>
-              <geometry>
-                  <box size="0.1 0.1 0.1"/>
-              </geometry>
-          </collision>
-          <visual>
-              <origin xyz="0 0 0" rpy="0 0 0"/>
-              <geometry>
-                  <box size="0.001 0.001 0.001"/>
-              </geometry>
-          </visual>
-          <inertial>
-              <mass value="1e-5"/>
-              <origin xyz="0 0 0" rpy="0 0 0"/>
-              <inertia ixx="1e-6" ixy="0" ixz="0" iyy="1e-6" iyz="0" izz="1e-6"/>
-          </inertial>
-      </link>
-      <joint name="$(arg asus_name)_joint" type="fixed">
-          <axis xyz="0 1 0"/>
-          <origin xyz="0.5 0 0.7" rpy="0 2.5 0"/> <!-- 0 2.5 0 -->
-          <!--        <origin xyz="0.5 0 0.7" rpy="0 3.14159 0"/>-->
-          <parent link="base_link"/>
-          <child link="$(arg asus_name)_base_link"/>
-      </joint>
-      <sensor_calibration_assembly sensor_id="$(arg asus_name)" parent_link="$(arg asus_name)_base_link"/>
+      <xacro:include filename="$(find asus_description)/urdf/asus/asus.xacro"/>
+      <asus_sensor parent="$(arg asus_name)_base_link" prefix="$(arg tf_prefix)/$(arg sensor_prefix)"  name="$(arg asus_name)"  cam_px="0" cam_py="0" cam_pz="0" cam_or="0" cam_op="0" cam_oy="0"/>
+      <sensor_calibration_assembly sensor_id="$(arg asus_name)" parent_link="base_link" final_link_suffix="base_link"/>
     </xacro:if>
 </robot>

Commit message: Fix transform of Velodyne, it is set by calibration files instead

File: base_simulation/urdf/iliad_uol_cititruck.xacro (robot description, xacro)
@@ -376,5 +376,5 @@
       <xacro:include filename="$(find velodyne_description8)/urdf/VLP-16.urdf.xacro"/>
       <VLP-16 parent="velodyne_base_link" gpu="true" name="velodyne" topic="/$(arg tf_prefix)/$(arg sensor_prefix)/velodyne/velodyne_points" hz="10" samples="440">
-          <origin xyz="0.8 0 0.95" rpy="0 0 0" />
+          <origin xyz="0 0 0" rpy="0 0 0" />
       </VLP-16>
      <sensor_calibration_assembly sensor_id="velodyne" parent_link="base_link" final_link_suffix="base_link"/>

Commit message: Timms modification of the initial position of the Kinect v2 sensor so it is easier to calibrate.

File: base_simulation/urdf/iliad_uol_cititruck.xacro (robot description, xacro)
@@ -374,21 +374,45 @@
     <!-- FIXED: The name should be velodyne_link -->
     <xacro:if value="$(arg velodyne)">
-      <xacro:include filename="$(find velodyne_description8)/urdf/VLP-16.urdf.xacro"/>
-      <VLP-16 parent="velodyne_base_link" gpu="true" name="velodyne" topic="/$(arg tf_prefix)/$(arg sensor_prefix)/velodyne/velodyne_points" hz="10" samples="440">
-          <origin xyz="0 0 0" rpy="0 0 0" />
+      <xacro:include filename="$(find velodyne_description)/urdf/VLP-16.urdf.xacro"/>
+      <VLP-16 parent="velodyne_base_link" prefix="$(arg tf_prefix)" name="velodyne_link" topic="$(arg sensor_prefix)/velodyne_points" hz="10" samples="440">
+          <origin xyz="0 0 0" rpy="0 0 0" /> <!-- given by calibration -->
       </VLP-16>
-     <sensor_calibration_assembly sensor_id="velodyne" parent_link="base_link" final_link_suffix="base_link"/>
+      <sensor_calibration_assembly sensor_id="velodyne" parent_link="base_link" final_link_suffix="base_link"/>
     </xacro:if>
     <!-- Kinect v2 -->
     <xacro:if value="$(arg kinect2)">
-    <xacro:include filename="$(find kinect2_description)/urdf/kinect2/kinect2.xacro"/>
+      <xacro:include filename="$(find kinect2_description)/urdf/kinect2/kinect2.xacro"/>
       <kinect2_sensor parent="kinect2_base_link" prefix="$(arg tf_prefix)/$(arg sensor_prefix)" name="kinect2" cam_px="0" cam_py="0" cam_pz="0" cam_or="0" cam_op="0" cam_oy="3.1415926"/>
       <sensor_calibration_assembly sensor_id="kinect2" parent_link="base_link" final_link_suffix="base_link"/>
     </xacro:if>
-    <!-- Asus for pallet detection -->
+    <!-- Asus for pallet detection (deprecated?) -->
     <xacro:if value="$(arg asus)">
-      <xacro:include filename="$(find asus_description)/urdf/asus/asus.xacro"/>
-      <asus_sensor parent="$(arg asus_name)_base_link" prefix="$(arg tf_prefix)/$(arg sensor_prefix)"  name="$(arg asus_name)"  cam_px="0" cam_py="0" cam_pz="0" cam_or="0" cam_op="0" cam_oy="0"/>
-      <sensor_calibration_assembly sensor_id="$(arg asus_name)" parent_link="base_link" final_link_suffix="base_link"/>
+      <link name="$(arg asus_name)_base_link">
+          <collision>
+              <origin xyz="0 0 0" rpy="0 0 0"/>
+              <geometry>
+                  <box size="0.1 0.1 0.1"/>
+              </geometry>
+          </collision>
+          <visual>
+              <origin xyz="0 0 0" rpy="0 0 0"/>
+              <geometry>
+                  <box size="0.001 0.001 0.001"/>
+              </geometry>
+          </visual>
+          <inertial>
+              <mass value="1e-5"/>
+              <origin xyz="0 0 0" rpy="0 0 0"/>
+              <inertia ixx="1e-6" ixy="0" ixz="0" iyy="1e-6" iyz="0" izz="1e-6"/>
+          </inertial>
+      </link>
+      <joint name="$(arg asus_name)_joint" type="fixed">
+          <axis xyz="0 1 0"/>
+          <origin xyz="0.5 0 0.7" rpy="0 2.5 0"/> <!-- 0 2.5 0 -->
+          <!--        <origin xyz="0.5 0 0.7" rpy="0 3.14159 0"/>-->
+          <parent link="base_link"/>
+          <child link="$(arg asus_name)_base_link"/>
+      </joint>
+      <sensor_calibration_assembly sensor_id="$(arg asus_name)" parent_link="$(arg asus_name)_base_link"/>
     </xacro:if>
 </robot>

Commit message: I commited the wrong file before

File: base_simulation/urdf/iliad_uol_cititruck.xacro (robot description, xacro)
@@ -374,45 +374,21 @@
     <!-- FIXED: The name should be velodyne_link -->
     <xacro:if value="$(arg velodyne)">
-      <xacro:include filename="$(find velodyne_description)/urdf/VLP-16.urdf.xacro"/>
-      <VLP-16 parent="velodyne_base_link" prefix="$(arg tf_prefix)" name="velodyne_link" topic="$(arg sensor_prefix)/velodyne_points" hz="10" samples="440">
-          <origin xyz="0 0 0" rpy="0 0 0" /> <!-- given by calibration -->
+      <xacro:include filename="$(find velodyne_description8)/urdf/VLP-16.urdf.xacro"/>
+      <VLP-16 parent="velodyne_base_link" gpu="true" name="velodyne" topic="/$(arg tf_prefix)/$(arg sensor_prefix)/velodyne/velodyne_points" hz="10" samples="440">
+          <origin xyz="0 0 0" rpy="0 0 0" />
       </VLP-16>
-      <sensor_calibration_assembly sensor_id="velodyne" parent_link="base_link" final_link_suffix="base_link"/>
+     <sensor_calibration_assembly sensor_id="velodyne" parent_link="base_link" final_link_suffix="base_link"/>
     </xacro:if>
     <!-- Kinect v2 -->
     <xacro:if value="$(arg kinect2)">
-      <xacro:include filename="$(find kinect2_description)/urdf/kinect2/kinect2.xacro"/>
-      <kinect2_sensor parent="kinect2_base_link" prefix="$(arg tf_prefix)/$(arg sensor_prefix)" name="kinect2" cam_px="0" cam_py="0" cam_pz="0" cam_or="0" cam_op="0" cam_oy="3.1415926"/>
+    <xacro:include filename="$(find kinect2_description)/urdf/kinect2/kinect2.xacro"/>
+      <kinect2_sensor parent="kinect2_base_link" prefix="$(arg tf_prefix)/$(arg sensor_prefix)" name="kinect2" cam_px="0" cam_py="0" cam_pz="0" cam_or="-1.5707" cam_op="0" cam_oy="-1.5707"/>
       <sensor_calibration_assembly sensor_id="kinect2" parent_link="base_link" final_link_suffix="base_link"/>
     </xacro:if>
-    <!-- Asus for pallet detection (deprecated?) -->
+    <!-- Asus for pallet detection -->
     <xacro:if value="$(arg asus)">
-      <link name="$(arg asus_name)_base_link">
-          <collision>
-              <origin xyz="0 0 0" rpy="0 0 0"/>
-              <geometry>
-                  <box size="0.1 0.1 0.1"/>
-              </geometry>
-          </collision>
-          <visual>
-              <origin xyz="0 0 0" rpy="0 0 0"/>
-              <geometry>
-                  <box size="0.001 0.001 0.001"/>
-              </geometry>
-          </visual>
-          <inertial>
-              <mass value="1e-5"/>
-              <origin xyz="0 0 0" rpy="0 0 0"/>
-              <inertia ixx="1e-6" ixy="0" ixz="0" iyy="1e-6" iyz="0" izz="1e-6"/>
-          </inertial>
-      </link>
-      <joint name="$(arg asus_name)_joint" type="fixed">
-          <axis xyz="0 1 0"/>
-          <origin xyz="0.5 0 0.7" rpy="0 2.5 0"/> <!-- 0 2.5 0 -->
-          <!--        <origin xyz="0.5 0 0.7" rpy="0 3.14159 0"/>-->
-          <parent link="base_link"/>
-          <child link="$(arg asus_name)_base_link"/>
-      </joint>
-      <sensor_calibration_assembly sensor_id="$(arg asus_name)" parent_link="$(arg asus_name)_base_link"/>
+      <xacro:include filename="$(find asus_description)/urdf/asus/asus.xacro"/>
+      <asus_sensor parent="$(arg asus_name)_base_link" prefix="$(arg tf_prefix)/$(arg sensor_prefix)"  name="$(arg asus_name)"  cam_px="0" cam_py="0" cam_pz="0" cam_or="0" cam_op="0" cam_oy="0"/>
+      <sensor_calibration_assembly sensor_id="$(arg asus_name)" parent_link="base_link" final_link_suffix="base_link"/>
     </xacro:if>
 </robot>
