Commit message: Corrected citi xacro to allow laser detections. Corrected actor xacro: lower gravity center of mass and laser closer to floor to easily detect pallets and such. Corrected teb parameters for slower human movement and wider avoidance of local obstacles.

File: iliad_base_simulation/urdf/iliad_uol_cititruck.xacro (robot description, xacro)
@@ -42,7 +42,7 @@
         </inertial>
         <collision>
-            <origin xyz="0.8 0 0.1" rpy="0 0 0"/>
-            <geometry>
-                <box size="0.4 0.55 0.005"/>
+            <origin xyz="0.8 0 0.4" rpy="0 0 0"/>
+            <geometry>
+                <box size="0.4 0.55 0.75"/>
             </geometry>
         </collision>

File: moving_actor_gazebo/urdf/actor_cpu.xacro (robot description, xacro)
@@ -14,4 +14,5 @@
       <odometryRate>20.0</odometryRate>
       <robotBaseFrame>$(arg tf_prefix)/base_footprint</robotBaseFrame>
+      <enableYAxis>1</enableYAxis>
     </plugin>
   </gazebo>
@@ -20,8 +21,21 @@
   <link name="$(arg tf_prefix)/base_link">
     <inertial>
+      <origin xyz="0.0 0.0 -0.85" rpy="0 0 0"/>
       <mass value="80"/>
       <inertia ixx="22.85" ixy="0.0" ixz="0.0" iyy="22.85" iyz="0.0" izz="2.5"/>
     </inertial>
-    <visual name="$(arg actor_name)_magic_carpet">
+    <collision name="$(arg actor_name)_collision">
+      <origin xyz="0 0 0.0" rpy="0.0 0 0"/>
+      <geometry>
+        <box size="0.5 0.5 1.8"/>
+      </geometry>
+    </collision>
+    <visual name="$(arg actor_name)_visual">
+      <origin xyz="0 0 -0.9" rpy="0.0 0 1.54"/>
+      <geometry>
+        <mesh filename="model://person_standing/meshes/standing.dae"/>
+      </geometry>
+    </visual>
+    <!-- <visual name="$(arg actor_name)_magic_carpet">
       <origin xyz="0 0 0.0" rpy="0.0 0 0"/>
       <geometry>
@@ -41,7 +55,10 @@
       </geometry>
     </visual>
+    -->
   </link>
   <gazebo reference="$(arg tf_prefix)/base_link">
     <selfCollide>false</selfCollide>
+    <mu1>0.02</mu1>
+    <mu2>0.02</mu2>
   </gazebo>
   <link name="$(arg tf_prefix)/hokuyo"/>
@@ -57,5 +74,5 @@
     <child link="$(arg tf_prefix)/hokuyo"/>
     <axis xyz="0 1 0" />
-    <origin xyz="0.175 0 0.73" rpy="0 0 0"/>
+    <origin xyz="0.27 0 -0.85" rpy="0 0 0"/>
   </joint>
   <!-- CREATE SENSORS -->

File: moving_actor_gazebo/urdf/actor_gpu.xacro (robot description, xacro)
@@ -14,4 +14,5 @@
       <odometryRate>20.0</odometryRate>
       <robotBaseFrame>$(arg tf_prefix)/base_footprint</robotBaseFrame>
+      <enableYAxis>1</enableYAxis>
     </plugin>
   </gazebo>
@@ -20,8 +21,21 @@
   <link name="$(arg tf_prefix)/base_link">
     <inertial>
+      <origin xyz="0.0 0.0 -0.85" rpy="0 0 0"/>
       <mass value="80"/>
       <inertia ixx="22.85" ixy="0.0" ixz="0.0" iyy="22.85" iyz="0.0" izz="2.5"/>
     </inertial>
-    <visual name="$(arg actor_name)_magic_carpet">
+    <collision name="$(arg actor_name)_collision">
+      <origin xyz="0 0 0.0" rpy="0.0 0 0"/>
+      <geometry>
+        <box size="0.5 0.5 1.8"/>
+      </geometry>
+    </collision>
+    <visual name="$(arg actor_name)_visual">
+      <origin xyz="0 0 -0.9" rpy="0.0 0 1.54"/>
+      <geometry>
+        <mesh filename="model://person_standing/meshes/standing.dae"/>
+      </geometry>
+    </visual>
+    <!-- <visual name="$(arg actor_name)_magic_carpet">
       <origin xyz="0 0 0.0" rpy="0.0 0 0"/>
       <geometry>
@@ -41,7 +55,10 @@
       </geometry>
     </visual>
+    -->
   </link>
   <gazebo reference="$(arg tf_prefix)/base_link">
     <selfCollide>false</selfCollide>
+    <mu1>0.02</mu1>
+    <mu2>0.02</mu2>
   </gazebo>
   <link name="$(arg tf_prefix)/hokuyo"/>
@@ -57,5 +74,5 @@
     <child link="$(arg tf_prefix)/hokuyo"/>
     <axis xyz="0 1 0" />
-    <origin xyz="0.175 0 0.73" rpy="0 0 0"/>
+    <origin xyz="0.27 0 -0.85" rpy="0 0 0"/>
   </joint>
   <!-- CREATE SENSORS -->

Commit message: added nodes and changes to evalute the safety layers and run experiemnts

File: iliad_base_simulation/urdf/iliad_uol_cititruck.xacro (robot description, xacro)
@@ -44,5 +44,5 @@
             <origin xyz="0.8 0 0.4" rpy="0 0 0"/>
             <geometry>
-                <box size="0.4 0.55 0.75"/>
+                <box size="0.4 0.55 0.80"/>
             </geometry>
         </collision>
